File: pcb/usb_cdc.sch (KiCad schematic (older format))
At the start: 23 parts

Commit message: digital schematic commit
Parts:
- added C? (x5): 1uF, symbol C
- added J?: RS232, symbol DB9
- added P?: I2C, symbol CONN_4
- added R? (x2): 2.2k, symbol R
- added U?: MAX232, symbol MAX232
Connections:
- net 3V3: now also P?.4 (P4), R?.1, R?.1
- net GND: now also C?.1, C?.1, C?.1, J?.5, P?.1 (P1), U?.15 (GND)
- net tem1_en: now reaches D?.10 (PC2)
- net tem1_dir: now reaches D?.11 (PC3)
- net usart2_cts: now reaches D?.14 (PA0)
- net usart2_cts: now also U?.9 (R2OUT)
- net usart2_rts: now reaches D?.15 (PA1)
- net usart2_rts: now also U?.10 (T2IN)
- net usart2_tx: now reaches D?.16 (PA2)
- net usart2_tx: now also U?.11 (T1IN)
- net usart2_rx: now reaches D?.17 (PA3)
- net usart2_rx: now also U?.12 (R1OUT)
- net tem2_en: now reaches D?.24 (PC4)
- net tem2_dir: now reaches D?.25 (PC5)
- net tem3_en: now reaches D?.37 (PC6)
- net tem3_dir: now reaches D?.38 (PC7)
- net usb_dm: now reaches D?.44 (PA11), R?.2
- net usb_dp: now reaches D?.45 (PA12), R?.2, R?.2
- net i2c1_scl: now reaches D?.58 (PB6)
- net i2c1_scl: now also P?.2 (P2), R?.2
- net i2c1_sda: now reaches D?.59 (PB7)
- net i2c1_sda: now also P?.3 (P3), R?.2
- net tem0_en: now reaches D?.8 (PC0)
- net tem0_dir: now reaches D?.9 (PC1)
- net +5V: now reaches J?.1 (Vbus), R?.2
- net +5V: now also C?.2, U?.16 (VCC)
- new net: C?.1, U?.1 (C1+)
- new net: J?.2, U?.13 (R1IN)
- new net: J?.3, U?.14 (T1OUT)
- new net: C?.2, U?.2 (V+)
- new net: C?.2, U?.3 (C1-)
- new net: C?.1, U?.4 (C2+)
- new net: C?.2, U?.5 (C2-)
- new net: C?.2, U?.6 (V-)
- new net: J?.7 (P7), U?.7 (T2OUT)
- new net: J?.8 (P8), U?.8 (R2IN)
Other:
- note added: "U\nS\nB\nL\nC\n6"
- moved on the sheet: C?, D?, J?, P?, Q?, R?, X?

Commit message: briges added
Parts:
- added C?: CP1, symbol CP1
- added C? (x7): C, symbol C
- added D? (x16): ZENER, symbol ZENER
- added D? (x16): DIODE, symbol DIODE
- added D? (x8): TLP181GB, symbol TLP181GB
- added D?: P6AU, symbol P6AU
- added F?: FUSE, symbol FUSE
- added P? (x5): CONN_2, symbol CONN_2
- added Q? (x16): MOSFET_N, symbol MOSFET_N
- added R? (x8): 2k, symbol R
- added R? (x8): 10k, symbol R
- added R? (x8): R, symbol R
- added U? (x12): 4001, symbol 4001
Connections:
- net +5V: now also C?.1, D?.2 (IN+)
- net GND: now also C?.2, D?.1 (IN-), D?.3, D?.3, D?.3, D?.3, D?.3, D?.3, D?.3, D?.3
- new net: D?.2 (K), D?.2 (K), Q?.G, Q?.G, R?.1 (x8)
- new net: D?.1 (A), D?.1 (A), D?.2 (K), P?.1 (P1), Q?.D (x4)
- new net: D?.1 (A), D?.1 (A), D?.2 (K), P?.2 (PM), Q?.D, Q?.S (x4)
- new net: F?.1, P?.2 (PM)
- new net: D?.6, R?.2, U?.1, U?.2 (x4)
- new net: D?.6, R?.2, U?.1, U?.2, U?.2 (x4)
- new net: R?.1, R?.2, U?.3 (x8)
- new net: U?.1, U?.3 (x4)
- new net +12V: C?.1, C?.1, D?.2 (K), D?.2 (K), D?.2 (K), D?.2 (K), D?.2 (K), D?.2 (K), D?.2 (K), D?.2 (K), F?.2, Q?.D, Q?.D, Q?.D, Q?.D, Q?.D, Q?.D, Q?.D, Q?.D
- new net GNDPWR: C?.2, C?.2, C?.2, D?.1 (A), D?.1 (A), D?.1 (A), D?.1 (A), D?.1 (A), D?.1 (A), D?.1 (A), D?.1 (A), D?.1 (A), D?.1 (A), D?.1 (A), D?.1 (A), D?.1 (A), D?.1 (A), D?.1 (A), D?.1 (A), D?.3 (OUT-), D?.4, D?.4, D?.4, D?.4, D?.4, D?.4, D?.4, D?.4, P?.1 (P1), Q?.S, Q?.S, Q?.S, Q?.S, Q?.S, Q?.S, Q?.S, Q?.S, R?.2, R?.2, R?.2, R?.2, R?.2, R?.2, R?.2, R?.2, U?.7 (VSS), U?.7 (VSS), U?.7 (VSS), U?.7 (VSS), U?.7 (VSS), U?.7 (VSS), U?.7 (VSS), U?.7 (VSS), U?.7 (VSS), U?.7 (VSS), U?.7 (VSS), U?.7 (VSS)
- new net VDD: C?.1, D?.4 (OUT+), R?.1, R?.1, R?.1, R?.1, R?.1, R?.1, R?.1, R?.1, U?.14 (VDD), U?.14 (VDD), U?.14 (VDD), U?.14 (VDD), U?.14 (VDD), U?.14 (VDD), U?.14 (VDD), U?.14 (VDD), U?.14 (VDD), U?.14 (VDD), U?.14 (VDD), U?.14 (VDD)
Other:
- note added: "dir"
- note added: "en"

Commit message: some changes
Parts:
- gave numbers to parts that had none: 131
Connections:
- net tem0_dir: now also D103.1
- net tem0_en: now also D104.1
- net tem1_dir: now also D105.1
- net tem1_en: now also D106.1
- net tem2_dir: now also D107.1
- net tem2_en: now also D108.1
- net tem3_dir: now also D109.1
- net tem3_en: now also D110.1
- net at J102.2 (D-): no longer R109.1
- net at J102.3 (D+): no longer R108.1
- net at Q103.S: now also D111.1 (A), D119.1 (A), D120.2 (K), P104.1 (P1), Q104.D
- net at D104.6, R110.2, U103.2: now also U103.5; no longer U103.1
- net at D103.6, R114.2, U102.1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: now also U103.6; no longer U103.2
- net at R118.1, R127.2: now also U103.4; no longer U103.3
- net at D106.6, R111.2: now also U103.12, U103.9; no longer U103.1, U103.2
- net at R119.1, R129.2: now also U103.11; no longer U103.3
- net at R123.1, R128.2: now also U103.10; no longer U103.3
- net at D113.1 (A), D121.1 (A), D122.2 (K)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: now also Q105.S
- net at Q109.S: now also D117.1 (A), D125.1 (A), D126.2 (K), P107.1 (P1), Q110.D
- net at D110.6, R113.2: now also U104.12, U104.9; no longer U104.1, U104.2
- net at R121.1, R133.2: now also U104.11; no longer U104.3
- net at R125.1, R132.2: now also U104.10; no longer U104.3
- net at D108.6, R112.2, U104.2: now also U104.5; no longer U104.1
- net at U104.1: now also U102.10; no longer U102.3
- net at R120.1, R131.2: now also U104.4; no longer U104.3
- net at D115.1 (A), D123.1 (A), D124.2 (K)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: now also Q107.S
- new net: D105.6, R115.2, U102.5, U102.6, U103.13
- new net: U102.4, U103.8
- new net: D109.6, R117.2, U102.12, U102.13, U104.13
- new net: U102.11, U104.8
- new net: D107.6, R116.2, U102.8, U102.9, U104.6
Other:
- note added: "15V"
- note added: "5V -> 15V"
- note removed: "dir"
- note removed: "en"
- moved on the sheet: C101, C102, C103, C104, C105, C106, C107, C108, C109, C110, C111, C112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
